File: led-tube.kicad_pcb (KiCad board)
At the start: 2 copper layers, 32 x 498 mm, 139 parts, among them Q1 RU20P7C_C605444, Q2 RU20P7C_C605444, Q3 RU20P7C_C605444, SW1 K2-1112SW-A4SW-04, SW2 K2-1112SW-A4SW-04, U1 QuinLED-ESP32, U10 19-217_R6C-AL1M2VY_3T, U11 SMTSO3015CTJ, U14 SMTSO3015CTJ, U15 SMTSO3015CTJ, U2 U262-161N-4BVC11, U3 IP5328P, U5 19-217_R6C-AL1M2VY_3T, U6 SN74AHCT32QPWRQ1, U7 19-217_R6C-AL1M2VY_3T, U8 19-217_R6C-AL1M2VY_3T, U9 19-217_R6C-AL1M2VY_3T

Commit message: place components, don't place leds but use ledstrips instead
Parts:
- removed BT3, BT4: BH-18650-B1BA002, easyeda2kicad:BATTERY-SMD_18650-1S-L77.1-W20.7-1
- removed C14, C41: 10uf, Capacitor_SMD:C_0603_1608Metric_Pad1.08x0.95mm_HandSolder
- removed C21, C22, C23, C24, C25, C26, C27, C28, C29, C30, C31, C32, C33, C34, C35, C36, C37, C53, C54, C55, C56, C57, C58, C59, C60, C61, C62: 0.1uF, Capacitor_SMD:C_0603_1608Metric_Pad1.08x0.95mm_HandSolder
- removed C38, C39, C40, C43, C45, C46, C47, C48: 22uf, Capacitor_SMD:C_0805_2012Metric_Pad1.18x1.45mm_HandSolder
- removed C42, C44: 100nf, Capacitor_SMD:C_0603_1608Metric_Pad1.08x0.95mm_HandSolder
- removed C49, C50: 2.2uf, Capacitor_SMD:C_0603_1608Metric_Pad1.08x0.95mm_HandSolder
- removed F2: BSMD1812-350-16V, easyeda2kicad:F1812
- removed LED1, LED10, LED11, LED12, LED13, LED14, LED15, LED16, LED17, LED18, LED19, LED2, LED20, LED21, LED22, LED23, LED24, LED25, LED26, LED27, LED28, LED29, LED3, LED30, LED31, LED32, LED33, LED34, LED35, LED36, LED37, LED38, LED39, LED4, LED40, LED5, LED6, LED7, LED8, LED9: XL-5050RGBC-WS2812B, LED_SMD:LED_WS2812B_PLCC4_5.0x5.0mm_P3.2mm
- removed Q3: RU20P7C_C605444, easyeda2kicad:SOT-23-3_L2.9-W1.6-P1.90-LS2.8-BR
- removed USB1: MICROXNJ, easyeda2kicad:MICRO-USB-SMD_MICROXNJ
- added C15: 1uF, Capacitor_SMD:C_0603_1608Metric_Pad1.08x0.95mm_HandSolder, F.Cu at (624.3, 544.0)
- added C16: 0.1uF, Capacitor_SMD:C_0603_1608Metric_Pad1.08x0.95mm_HandSolder, F.Cu at (625.8, 544.0)
- added F1: BSMD2920-500-16V, easyeda2kicad:F2920, F.Cu at (616.0, 521.2)
- added JP1: SolderJumper_2_Bridged, Jumper:SolderJumper-2_P1.3mm_Bridged_RoundedPad1.0x1.5mm, F.Cu at (624.5, 540.7)
- added MIC1: MP34DT05TR-A, easyeda2kicad:MIC-SMD_5P-L3.0-W4.0-P0.85-BL, F.Cu at (629.0, 544.2)
- added P1: WJ15EDGRC-3.81-3P, easyeda2kicad:CONN-TH_3P-P3.81_WJ15EDGRC-3.81-3P, F.Cu at (615.9, 408.0)
- added R14: 100, Resistor_SMD:R_0603_1608Metric_Pad0.98x0.95mm_HandSolder, F.Cu at (601.8, 454.0)
- added R15: 100, Resistor_SMD:R_0603_1608Metric_Pad0.98x0.95mm_HandSolder, F.Cu at (602.7, 470.3)
- added SW3: K2-1112SW-A4SW-04, easyeda2kicad:KEY-TH_K2-1112SW-AXXW-XX, F.Cu at (601.9, 476.9)
- added SW4: SS-12M11G5, easyeda2kicad:SW-TH_XKB_SS-12M11XX, F.Cu at (628.3, 508.0)
- added U4: 19-217_R6C-AL1M2VY_3T, footprint:LED0603-R-RD, F.Cu at (629.7, 476.0)
- BT1: moved to F.Cu
- C10, C11, C17, C18, C19, C20, C5, C8: value 0.1uF -> 22uf; footprint Capacitor_SMD:C_0603_1608Metric_Pad1.08x0.95mm_HandSolder -> Capacitor_SMD:C_0805_2012Metric_Pad1.18x1.45mm_HandSolder
- C12: value 100nf -> 22uf; footprint Capacitor_SMD:C_0603_1608Metric_Pad1.08x0.95mm_HandSolder -> Capacitor_SMD:C_0805_2012Metric_Pad1.18x1.45mm_HandSolder
- C13: value 22uf -> 10uf; footprint Capacitor_SMD:C_0805_2012Metric_Pad1.18x1.45mm_HandSolder -> Capacitor_SMD:C_0603_1608Metric_Pad1.08x0.95mm_HandSolder
- C3, C4: value 0.1uF -> 2.2uf
- C6, C7, C9: value 0.1uF -> 100nf
- R11, R12: moved to B.Cu
- R13: value 10k -> 100
- R2: value 113k -> 10k
- R4: value 100 -> 82k
- R5: value 100 -> 113k
- R8: value 82k -> 100
- U10: value 19-217_R6C-AL1M2VY_3T -> SMTSO3015CTJ; footprint footprint:LED0603-R-RD -> footprint:SMTSO3030CTJ
- U3: value IP5328P -> 19-217_R6C-AL1M2VY_3T; footprint easyeda2kicad:QFN-40_L6.0-W6.0-P0.50-BL-EP -> footprint:LED0603-R-RD
- U5: value 19-217_R6C-AL1M2VY_3T -> IP5328P; footprint footprint:LED0603-R-RD -> easyeda2kicad:QFN-40_L6.0-W6.0-P0.50-BL-EP
- moved C5 699.6 mm to (607.6, 529.8), turned to 90 degrees
- moved C6 693.2 mm to (609.4, 530.0), turned to 90 degrees
- moved C10 680.0 mm to (608.5, 523.3), turned to 180 degrees
- moved C7 674.8 mm to (608.5, 527.1)
- moved C9 672.0 mm to (615.1, 527.4), turned to 180 degrees
- moved C4 663.6 mm to (613.1, 538.7)
- moved C11 655.3 mm to (608.5, 521.3), turned to 180 degrees
- moved C8 643.2 mm to (608.5, 525.3), turned to 180 degrees
- moved C18 593.7 mm to (607.7, 498.5), turned to 90 degrees
- moved C19 578.2 mm to (605.7, 498.5), turned to 90 degrees
- moved C3 575.0 mm to (608.1, 533.3)
- moved C20 570.0 mm to (603.7, 498.5), turned to 90 degrees
- moved C17 553.8 mm to (609.7, 498.5), turned to 90 degrees
- moved U11 490.2 mm to (604.0, 545.7)
- moved U15 348.8 mm to (603.9, 404.1)
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Connections:
- C10 pad 1: GND -> VSYS
- C10 pad 2: +5V -> GND
- C11 pad 1: GND -> VSYS
- C11 pad 2: +5V -> GND
- C12 pad 1: GND -> VSYS
- C12 pad 2: VSYS -> GND
- C17 pad 1: GND -> VBAT
- C17 pad 2: +5V -> GND
- C18 pad 1: GND -> VBAT
- C18 pad 2: +5V -> GND
- C19 pad 1: GND -> VBAT
- C19 pad 2: +5V -> GND
- C20 pad 1: GND -> VBAT
- C20 pad 2: +5V -> GND
- C3 pad 2: +5V -> VBAT
- C4 pad 1: GND -> VREG
- C4 pad 2: +5V -> GND
- C5 pad 1: GND -> VMID
- C5 pad 2: +5V -> GND
- C6 pad 1: GND -> VMID
- C6 pad 2: +5V -> GND
- C7 pad 2: +5V -> VSYS
- C8 pad 1: GND -> VSYS
- C8 pad 2: +5V -> GND
- C9 pad 1: GND -> Net-(C9-Pad1)
- C9 pad 2: +5V -> Net-(U5-BST)
- L1 pad 1: Net-(C44-Pad1) -> Net-(C9-Pad1)
- R13 pad 1: Net-(U3-VOUT2) -> GND
- R13 pad 2: VREG -> Net-(U3-A)
- R2 pad 1: Net-(U3-RSET) -> Net-(U5-VOUT2)
- R2 pad 2: GND -> VREG
- R4 pad 1: Net-(U3-LIGHT) -> GND
- R4 pad 2: Net-(U5-A) -> Net-(U5-NTC)
- R5 pad 1: Net-(U3-L1) -> Net-(U5-RSET)
- R5 pad 2: Net-(U10-A) -> GND
- R6 pad 1: Net-(U3-L2) -> Net-(U5-L1)
- R6 pad 2: Net-(U7-A) -> Net-(U3-C)
- R7 pad 1: GND -> Net-(U5-L2)
- R7 pad 2: Net-(U10-C) -> Net-(U4-C)
- R8 pad 1: GND -> Net-(U5-LIGHT)
- R8 pad 2: Net-(U3-NTC) -> Net-(U8-A)
- RT1 pad 1: Net-(U3-NTC) -> Net-(U5-NTC)
- U1 pad 17: unconnected-(U1-3v3-Pad17) -> +3.3V
- U1 pad 31: unconnected-(U1-IO32-Pad31) -> IO32/MIC DATA
- U1 pad 32: unconnected-(U1-IO12-Pad32) -> IO12/MIC CLK
- U10 pad 1: Net-(U10-A) -> GND
- U15 pad 1: LED DATA NEXT BOARD -> LED DATA OUT
- U3 pad 1: unconnected-(U3-DPA2-Pad1) -> Net-(U3-A)
- U3 pad 2: USB-C CC1 -> Net-(U3-C)
- U5 pad 1: Net-(U5-A) -> unconnected-(U5-DPA2-Pad1)
- U5 pad 2: GND -> USB-C CC1
- U7 pad 1: Net-(U7-A) -> Net-(U3-C)
- U7 pad 2: Net-(U10-C) -> Net-(U3-A)
- U8 pad 1: Net-(U10-C) -> Net-(U8-A)
- U8 pad 2: Net-(U7-A) -> GND
- U9 pad 1: Net-(U10-C) -> Net-(U4-C)
- U9 pad 2: Net-(U10-A) -> Net-(U3-A)
Routing:
- net +5V: track 0.00 -> 213.6 mm
- net GND: track 0.00 -> 164.7 mm, vias 0 -> 7
- net LED DATA OUT: track 0.00 -> 154.3 mm, vias 0 -> 1
- net KEY: track 0.00 -> 114.4 mm, vias 0 -> 2
- net VBAT: track 0.00 -> 110.5 mm, vias 0 -> 2
- net IO33/MAINBUTTON: track 0.00 -> 84.2 mm, vias 0 -> 1
- net Net-(U5-L2): track 0.00 -> 72.2 mm, vias 0 -> 2
- net Net-(U3-A): track 0.00 -> 64.9 mm, vias 0 -> 2
- net IO34/SECOND BUTTON: track 0.00 -> 62.9 mm, vias 0 -> 1
- net Net-(U5-LIGHT): track 0.00 -> 52.1 mm, vias 0 -> 2
- net VBUS: track 0.00 -> 48.3 mm
- net Net-(U5-L1): track 0.00 -> 44.4 mm, vias 0 -> 2
- net VSYS: track 0.00 -> 42.3 mm, vias 0 -> 2
- net +3.3V: track 0.00 -> 32.9 mm, vias 0 -> 1
- net VOUT1: track 0.00 -> 26.3 mm, vias 0 -> 2
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- added copper zone on B.Cu, net GND
- added copper zone on F.Cu, net GND
Other:
- board size 32 x 498 mm -> 32 x 150 mm

Commit message: add opensource hardware logo
Parts:
- added JP2: SolderJumper_2_Bridged, Jumper:SolderJumper-2_P1.3mm_Bridged_RoundedPad1.0x1.5mm, F.Cu at (607.7, 408.0)
Connections:
- U15 pad 1: LED DATA OUT -> Net-(JP2-B)
Routing:
- net Net-(JP2-B): track 0.00 -> 22.0 mm
- net LED DATA OUT: track 154.3 -> 133.7 mm
Other:
- board text added: "led-tube v0.1 github.com/janekc"
